Commit message: adjust to franka_robot_description

File: franka_robot_description/robots/common/franka_arm.srdf.xacro (robot description, xacro)
@@ -3,5 +3,5 @@
     <xacro:macro name="franka_arm_srdf" params="arm_id hand:='true' ee_id:=franka_hand arm_prefix='' no_prefix='false'">
         <xacro:property name="prefix" value="${'' if no_prefix else arm_prefix + arm_id + '_'}" />
-        <xacro:include filename="$(find franka_description)/robots/common/group_definition.xacro"/>
+        <xacro:include filename="$(find franka_robot_description)/robots/common/group_definition.xacro"/>
         <xacro:group_definition prefix="${prefix}" group_name="${prefix}arm" tip_link="${prefix}link8"/>
         <virtual_joint name="virtual_joint" type="fixed" parent_frame="world" child_link="base"/>
@@ -31,5 +31,5 @@
         <xacro:if value="${hand}">
             <xacro:if value="${ee_id == 'franka_hand'}">
-                <xacro:include filename="$(find franka_description)/end_effectors/franka_hand/franka_hand.srdf.xacro"/>
+                <xacro:include filename="$(find franka_robot_description)/end_effectors/franka_hand/franka_hand.srdf.xacro"/>
                 <xacro:franka_hand_srdf prefix="${prefix}"/>
             </xacro:if>

File: franka_robot_description/robots/common/franka_arm.xacro (robot description, xacro)
@@ -1,12 +1,12 @@
 <?xml version='1.0' encoding='utf-8'?>
 <robot xmlns:xacro="http://www.ros.org/wiki/xacro" name="franka_arm">
-  <xacro:include filename="$(find franka_description)/robots/common/utils.xacro" />
+  <xacro:include filename="$(find franka_robot_description)/robots/common/utils.xacro" />
   <!-- safety_distance: Minimum safety distance in [m] by which the collision volumes are expanded and which is enforced during robot motions -->
   <!-- arm_id: Namespace of the robot arm. Serves to differentiate between arms in case of multiple instances. -->
-  <!-- joint_limits: description of the joint limits that comes from a YAML file. Example definition: ${xacro.load_yaml('$(find franka_description)/robots/fr3/joint_limits.yaml')} -->
-  <!-- kinematics: description of the kinematics that comes from a YAML file. Example definition: ${xacro.load_yaml('$(find franka_description)/robots/fr3/kinematics.yaml')} -->
-  <!-- inertials: description of the inertials that comes from a YAML file. Example definition: ${xacro.load_yaml('$(find franka_description)/robots/fr3/inertials.yaml')} -->
-  <!-- dynamics: description of the dynamics that comes from a YAML file. Example definition: ${xacro.load_yaml('$(find franka_description)/robots/fr3/dynamics.yaml')} -->
-  <xacro:macro name="franka_arm" params="arm_id arm_prefix:='' no_prefix:=false description_pkg:='franka_description' connected_to:='base' xyz:='0 0 0' rpy:='0 0 0' gazebo:='false' safety_distance:=0 joint_limits inertials kinematics dynamics with_sc:=false" >
+  <!-- joint_limits: description of the joint limits that comes from a YAML file. Example definition: ${xacro.load_yaml('$(find franka_robot_description)/robots/fr3/joint_limits.yaml')} -->
+  <!-- kinematics: description of the kinematics that comes from a YAML file. Example definition: ${xacro.load_yaml('$(find franka_robot_description)/robots/fr3/kinematics.yaml')} -->
+  <!-- inertials: description of the inertials that comes from a YAML file. Example definition: ${xacro.load_yaml('$(find franka_robot_description)/robots/fr3/inertials.yaml')} -->
+  <!-- dynamics: description of the dynamics that comes from a YAML file. Example definition: ${xacro.load_yaml('$(find franka_robot_description)/robots/fr3/dynamics.yaml')} -->
+  <xacro:macro name="franka_arm" params="arm_id arm_prefix:='' no_prefix:=false description_pkg:='franka_robot_description' connected_to:='base' xyz:='0 0 0' rpy:='0 0 0' gazebo:='false' safety_distance:=0 joint_limits inertials kinematics dynamics with_sc:=false" >
     <!-- Define a property that defaults to 'arm_prefix_arm_id' concatenated with an underscore if 'no_prefix' is not set -->
     <xacro:property name="prefix" value="${'' if no_prefix else arm_prefix + arm_id + '_'}" />

File: franka_robot_description/robots/common/franka_robot.xacro (robot description, xacro)
@@ -27,8 +27,8 @@
                       no_prefix:='false'
                       arm_prefix:=''
-                      description_pkg:='franka_description'
+                      description_pkg:='franka_robot_description'
                       connected_to:='base'">
-    <xacro:include filename="$(find franka_description)/robots/common/utils.xacro" />
-    <xacro:include filename="$(find franka_description)/robots/common/franka_arm.xacro" />
+    <xacro:include filename="$(find franka_robot_description)/robots/common/utils.xacro" />
+    <xacro:include filename="$(find franka_robot_description)/robots/common/franka_arm.xacro" />
     <xacro:franka_arm
       arm_id="${arm_id}"
@@ -47,6 +47,6 @@
     />
     <xacro:if value="${hand and ee_id == 'franka_hand'}">
-      <xacro:include filename="$(find franka_description)/end_effectors/common/franka_hand.xacro"/>
-      <xacro:include filename="$(find franka_description)/end_effectors/common/utils.xacro" />
+      <xacro:include filename="$(find franka_robot_description)/end_effectors/common/franka_hand.xacro"/>
+      <xacro:include filename="$(find franka_robot_description)/end_effectors/common/utils.xacro" />
       <xacro:if value="${arm_id == 'fp3'}">
         <xacro:property name="ee_color" value="black" />
@@ -61,5 +61,5 @@
         arm_prefix="${arm_prefix}"
         ee_id="${ee_id}_${ee_color}"
-        ee_inertials="${xacro.load_yaml('$(find franka_description)/end_effectors/' + ee_id + '/inertials.yaml')}"
+        ee_inertials="${xacro.load_yaml('$(find franka_robot_description)/end_effectors/' + ee_id + '/inertials.yaml')}"
         rpy_ee="${rpy_ee}"
         xyz_ee="${xyz_ee}"
@@ -73,6 +73,6 @@
     </xacro:if>
     <xacro:if value="${hand and ee_id != 'none' and ee_id != 'franka_hand'}">
-      <xacro:include filename="$(find franka_description)/end_effectors/common/ee_with_one_link.xacro"/>
-      <xacro:include filename="$(find franka_description)/end_effectors/common/utils.xacro" />
+      <xacro:include filename="$(find franka_robot_description)/end_effectors/common/ee_with_one_link.xacro"/>
+      <xacro:include filename="$(find franka_robot_description)/end_effectors/common/utils.xacro" />
       <xacro:property name="connection" value="${special_connection if special_connection != '' else arm_id + '_link8'}" />
       <xacro:ee_with_one_link
@@ -81,5 +81,5 @@
         arm_prefix="${arm_prefix}"
         ee_id="${ee_id}"
-        ee_inertials="${xacro.load_yaml('$(find franka_description)/end_effectors/' + ee_id + '/inertials.yaml')}"
+        ee_inertials="${xacro.load_yaml('$(find franka_robot_description)/end_effectors/' + ee_id + '/inertials.yaml')}"
         rpy_ee="${rpy_ee}"
         xyz_ee="${xyz_ee}"
@@ -140,5 +140,5 @@
     </xacro:if>
     <xacro:if value="${ros2_control}">
-      <xacro:include filename="$(find franka_description)/robots/common/franka_arm.ros2_control.xacro"/>
+      <xacro:include filename="$(find franka_robot_description)/robots/common/franka_arm.ros2_control.xacro"/>
       <xacro:franka_arm_ros2_control
           arm_id="${arm_id}"

File: franka_robot_description/robots/common/utils.xacro (robot description, xacro)
@@ -38,10 +38,10 @@
       <visual name="${prefix}${name}_visual">
         <geometry>
-          <mesh filename="package://${description_pkg}/meshes/robot_arms/${arm_id}/visual/${name}.dae" />
+          <mesh filename="package://${description_pkg}/meshes/robots/${arm_id}/visual/${name}.dae" />
         </geometry>
       </visual>
       <collision name="${prefix}${name}_collision">
         <geometry>
-          <mesh filename="package://franka_description/meshes/robot_arms/${arm_id}/collision/${name}.stl" />
+          <mesh filename="package://franka_robot_description/meshes/robots/${arm_id}/collision/${name}.stl" />
         </geometry>
       </collision>

File: franka_robot_description/robots/fr3/fr3.srdf.xacro (robot description, xacro)
@@ -1,5 +1,5 @@
 <?xml version='1.0' encoding='utf-8'?>
 <robot xmlns:xacro="http://www.ros.org/wiki/xacro" name="fr3">
-  <xacro:include filename="$(find franka_description)/robots/common/franka_arm.srdf.xacro"/>
+  <xacro:include filename="$(find franka_robot_description)/robots/common/franka_arm.srdf.xacro"/>
   <!--
     DEPRECATION NOTICE

File: franka_robot_description/robots/fr3/fr3.urdf.xacro (robot description, xacro)
@@ -1,5 +1,5 @@
 <?xml version='1.0' encoding='utf-8'?>
 <robot xmlns:xacro="http://www.ros.org/wiki/xacro" name="fr3">
-  <xacro:include filename="$(find franka_description)/robots/common/franka_robot.xacro"/>
+  <xacro:include filename="$(find franka_robot_description)/robots/common/franka_robot.xacro"/>
   <!--
     DEPRECATION NOTICE
@@ -47,13 +47,13 @@
   <xacro:arg name="gazebo_effort" default="false" />
   <!-- Name of the description package -->
-  <xacro:arg name="description_pkg" default="franka_description" />
+  <xacro:arg name="description_pkg" default="franka_robot_description" />
   <!-- Append an underscore to the user-provided prefix, if non-empty. -->
   <xacro:property name="prefix" value="$(arg arm_prefix)"/>
   <xacro:property name="modified_prefix" value="${prefix + '_' if prefix else ''}"/>
   <xacro:franka_robot arm_id="fr3"
-                      joint_limits="${xacro.load_yaml('$(find franka_description)/robots/fr3/joint_limits.yaml')}"
-                      inertials="${xacro.load_yaml('$(find franka_description)/robots/fr3/inertials.yaml')}"
-                      kinematics="${xacro.load_yaml('$(find franka_description)/robots/fr3/kinematics.yaml')}"
-                      dynamics="${xacro.load_yaml('$(find franka_description)/robots/fr3/dynamics.yaml')}"
+                      joint_limits="${xacro.load_yaml('$(find franka_robot_description)/robots/fr3/joint_limits.yaml')}"
+                      inertials="${xacro.load_yaml('$(find franka_robot_description)/robots/fr3/inertials.yaml')}"
+                      kinematics="${xacro.load_yaml('$(find franka_robot_description)/robots/fr3/kinematics.yaml')}"
+                      dynamics="${xacro.load_yaml('$(find franka_robot_description)/robots/fr3/dynamics.yaml')}"
                       gazebo="$(arg gazebo)"
                       hand="$(arg hand)"

File: franka_robot_description/urdf/end_effectors/franka_hand/franka_hand.urdf.xacro (robot description, xacro)
@@ -1,11 +1,11 @@
 <?xml version="1.0" encoding="utf-8"?>
 <robot xmlns:xacro="http://www.ros.org/wiki/xacro" name="franka_hand">
-  <xacro:include filename="$(find franka_description)/end_effectors/common/utils.xacro" />
-  <xacro:include filename="$(find franka_description)/end_effectors/common/franka_hand.xacro"/>
-  <xacro:include filename="$(find franka_description)/end_effectors/franka_hand/franka_hand_arguments.xacro"/>
+  <xacro:include filename="$(find franka_robot_description)/end_effectors/common/utils.xacro" />
+  <xacro:include filename="$(find franka_robot_description)/end_effectors/common/franka_hand.xacro"/>
+  <xacro:include filename="$(find franka_robot_description)/end_effectors/franka_hand/franka_hand_arguments.xacro"/>
   <xacro:franka_hand connected_to="$(arg special_connection)"
                      arm_id="$(arg arm_id)"
                      ee_id="$(arg ee_id)_$(arg ee_color)"
-                     ee_inertials="${xacro.load_yaml('$(find franka_description)/end_effectors/$(arg ee_id)/inertials.yaml')}"
+                     ee_inertials="${xacro.load_yaml('$(find franka_robot_description)/end_effectors/$(arg ee_id)/inertials.yaml')}"
                      rpy_ee="$(arg rpy_ee)"
                      xyz_ee="$(arg xyz_ee)"

File: franka_robot_description/urdf/end_effectors/franka_hand/franka_hand_arguments.xacro (robot description, xacro)
@@ -24,4 +24,4 @@
   <xacro:arg name="gazebo" default="false" />
   <!-- Name of the description package -->
-  <xacro:arg name="description_pkg" default="franka_description" />
+  <xacro:arg name="description_pkg" default="franka_robot_description" />
 </robot>

File: franka_robot_description/urdf/main_assemblies/bimanual_dfki.urdf.xacro (robot description, xacro)
@@ -40,5 +40,5 @@
   <xacro:arg name="gazebo_effort" default="false" />
   <!-- Name of the description package -->
-  <xacro:arg name="description_pkg" default="franka_description" />
+  <xacro:arg name="description_pkg" default="franka_robot_description" />
   <xacro:arg name="gripper_type" default="franka_default" />
   <xacro:arg name="use_sim" default="false" />
@@ -46,5 +46,5 @@
   <xacro:property name="prefix" value="$(arg arm_prefix)"/>
   <xacro:property name="modified_prefix" value="${prefix + '_' if prefix else ''}"/>
-  <xacro:include filename="$(find franka_description)/robots/common/franka_robot.xacro"/>
+  <xacro:include filename="$(find franka_robot_description)/robots/common/franka_robot.xacro"/>
   <!-- <xacro:property name="arg_hand" value="$(arg hand)"/> -->
   <!-- <xacro:property name="arg_gripper_type" value="$(arg gripper_type)"/> -->
@@ -54,8 +54,8 @@
   <xacro:franka_robot
       arm_id="$(arg arm_id)"
-      joint_limits="${xacro.load_yaml('$(find franka_description)/robots/$(arg arm_id)/joint_limits.yaml')}"
-      inertials="${xacro.load_yaml('$(find franka_description)/robots/$(arg arm_id)/inertials.yaml')}"
-      kinematics="${xacro.load_yaml('$(find franka_description)/robots/$(arg arm_id)/kinematics.yaml')}"
-      dynamics="${xacro.load_yaml('$(find franka_description)/robots/$(arg arm_id)/dynamics.yaml')}"
+      joint_limits="${xacro.load_yaml('$(find franka_robot_description)/robots/$(arg arm_id)/joint_limits.yaml')}"
+      inertials="${xacro.load_yaml('$(find franka_robot_description)/robots/$(arg arm_id)/inertials.yaml')}"
+      kinematics="${xacro.load_yaml('$(find franka_robot_description)/robots/$(arg arm_id)/kinematics.yaml')}"
+      dynamics="${xacro.load_yaml('$(find franka_robot_description)/robots/$(arg arm_id)/dynamics.yaml')}"
       gazebo="$(arg gazebo)"
       hand="$(arg hand)"

File: franka_robot_description/urdf/robots/fr3/fr3.urdf.xacro (robot description, xacro)
@@ -25,5 +25,5 @@
   <xacro:property name="use_franka_hand" value="${'true' if '$(arg gripper_type)' == 'franka_default' else 'false'}" />
   <!-- Include franka_robot macro -->
-  <xacro:include filename="$(find franka_description)/robots/common/franka_robot.xacro"/>
+  <xacro:include filename="$(find franka_robot_description)/robots/common/franka_robot.xacro"/>
   <!-- ============================================== -->
   <!-- Base Robot Arm Instantiation                   -->
@@ -31,8 +31,8 @@
   <xacro:franka_robot
       arm_id="$(arg arm_id)"
-      joint_limits="${xacro.load_yaml('$(find franka_description)/robots/$(arg arm_id)/joint_limits.yaml')}"
-      inertials="${xacro.load_yaml('$(find franka_description)/robots/$(arg arm_id)/inertials.yaml')}"
-      kinematics="${xacro.load_yaml('$(find franka_description)/robots/$(arg arm_id)/kinematics.yaml')}"
-      dynamics="${xacro.load_yaml('$(find franka_description)/robots/$(arg arm_id)/dynamics.yaml')}"
+      joint_limits="${xacro.load_yaml('$(find franka_robot_description)/robots/$(arg arm_id)/joint_limits.yaml')}"
+      inertials="${xacro.load_yaml('$(find franka_robot_description)/robots/$(arg arm_id)/inertials.yaml')}"
+      kinematics="${xacro.load_yaml('$(find franka_robot_description)/robots/$(arg arm_id)/kinematics.yaml')}"
+      dynamics="${xacro.load_yaml('$(find franka_robot_description)/robots/$(arg arm_id)/dynamics.yaml')}"
       gazebo="$(arg gazebo)"
       hand="${use_franka_hand}"
