Commit message: fix paths and add the final main assembly

File: franka_robot_description/robots/common/franka_arm.srdf.xacro (robot description, xacro)
@@ -31,5 +31,5 @@
         <xacro:if value="${hand}">
             <xacro:if value="${ee_id == 'franka_hand'}">
-                <xacro:include filename="$(find franka_robot_description)/end_effectors/franka_hand/franka_hand.srdf.xacro"/>
+                <xacro:include filename="$(find franka_robot_description)/urdf/end_effectors/franka_hand/franka_hand.srdf.xacro"/>
                 <xacro:franka_hand_srdf prefix="${prefix}"/>
             </xacro:if>

File: franka_robot_description/robots/common/franka_robot.xacro (robot description, xacro)
@@ -47,6 +47,6 @@
     />
     <xacro:if value="${hand and ee_id == 'franka_hand'}">
-      <xacro:include filename="$(find franka_robot_description)/end_effectors/common/franka_hand.xacro"/>
-      <xacro:include filename="$(find franka_robot_description)/end_effectors/common/utils.xacro" />
+      <xacro:include filename="$(find franka_robot_description)/urdf/end_effectors/common/franka_hand.xacro"/>
+      <xacro:include filename="$(find franka_robot_description)/urdf/end_effectors/common/utils.xacro" />
       <xacro:if value="${arm_id == 'fp3'}">
         <xacro:property name="ee_color" value="black" />
@@ -61,5 +61,5 @@
         arm_prefix="${arm_prefix}"
         ee_id="${ee_id}_${ee_color}"
-        ee_inertials="${xacro.load_yaml('$(find franka_robot_description)/end_effectors/' + ee_id + '/inertials.yaml')}"
+        ee_inertials="${xacro.load_yaml('$(find franka_robot_description)/urdf/end_effectors/' + ee_id + '/inertials.yaml')}"
         rpy_ee="${rpy_ee}"
         xyz_ee="${xyz_ee}"
@@ -73,6 +73,6 @@
     </xacro:if>
     <xacro:if value="${hand and ee_id != 'none' and ee_id != 'franka_hand'}">
-      <xacro:include filename="$(find franka_robot_description)/end_effectors/common/ee_with_one_link.xacro"/>
-      <xacro:include filename="$(find franka_robot_description)/end_effectors/common/utils.xacro" />
+      <xacro:include filename="$(find franka_robot_description)/urdf/end_effectors/common/ee_with_one_link.xacro"/>
+      <xacro:include filename="$(find franka_robot_description)/urdf/end_effectors/common/utils.xacro" />
       <xacro:property name="connection" value="${special_connection if special_connection != '' else arm_id + '_link8'}" />
       <xacro:ee_with_one_link
@@ -81,5 +81,5 @@
         arm_prefix="${arm_prefix}"
         ee_id="${ee_id}"
-        ee_inertials="${xacro.load_yaml('$(find franka_robot_description)/end_effectors/' + ee_id + '/inertials.yaml')}"
+        ee_inertials="${xacro.load_yaml('$(find franka_robot_description)/urdf/end_effectors/' + ee_id + '/inertials.yaml')}"
         rpy_ee="${rpy_ee}"
         xyz_ee="${xyz_ee}"

File: franka_robot_description/urdf/end_effectors/franka_hand/franka_hand.urdf.xacro (robot description, xacro)
@@ -1,11 +1,11 @@
 <?xml version="1.0" encoding="utf-8"?>
 <robot xmlns:xacro="http://www.ros.org/wiki/xacro" name="franka_hand">
-  <xacro:include filename="$(find franka_robot_description)/end_effectors/common/utils.xacro" />
-  <xacro:include filename="$(find franka_robot_description)/end_effectors/common/franka_hand.xacro"/>
-  <xacro:include filename="$(find franka_robot_description)/end_effectors/franka_hand/franka_hand_arguments.xacro"/>
+  <xacro:include filename="$(find franka_robot_description)/urdf/end_effectors/common/utils.xacro" />
+  <xacro:include filename="$(find franka_robot_description)/urdf/end_effectors/common/franka_hand.xacro"/>
+  <xacro:include filename="$(find franka_robot_description)/urdf/end_effectors/franka_hand/franka_hand_arguments.xacro"/>
   <xacro:franka_hand connected_to="$(arg special_connection)"
                      arm_id="$(arg arm_id)"
                      ee_id="$(arg ee_id)_$(arg ee_color)"
-                     ee_inertials="${xacro.load_yaml('$(find franka_robot_description)/end_effectors/$(arg ee_id)/inertials.yaml')}"
+                     ee_inertials="${xacro.load_yaml('$(find franka_robot_description)/urdf/end_effectors/$(arg ee_id)/inertials.yaml')}"
                      rpy_ee="$(arg rpy_ee)"
                      xyz_ee="$(arg xyz_ee)"

File: franka_robot_description/urdf/main_assemblies/bimanual_dfki.urdf.xacro (robot description, xacro)
@@ -1,55 +1,42 @@
 <?xml version='1.0' encoding='utf-8'?>
-<robot xmlns:xacro="http://www.ros.org/wiki/xacro" name="franka">
+<robot xmlns:xacro="http://www.ros.org/wiki/xacro" name="fr3">
+  <!-- ============================================== -->
+  <!-- Arguments provided by franka.launch.py (YAML)  -->
+  <!-- ============================================== -->
   <xacro:arg name="arm_id" default="fr3" />
+  <xacro:arg name="robot_ip" default="" />
+  <xacro:arg name="use_fake_hardware" default="false" />
+  <xacro:arg name="fake_sensor_commands" default="false" />
+  <xacro:arg name="use_sim" default="false" />
   <xacro:arg name="arm_prefix" default="" />
-  <!-- Don't print a prefix for joints, visuals, and links? -->
-  <xacro:arg name="no_prefix" default="false"/>
-  <!-- Should an end-effector be mounted at the flange?" -->
-  <xacro:arg name="hand" default="false" />
-  <!-- Which end-effector would be mounted at the flange?" -->
-  <xacro:arg name="ee_id" default="franka_hand" />
-  <!-- Where is the end-effector connected to, if different from the robot flange?  -->
-  <xacro:arg name="special_connection" default="" />
-  <!-- Position offset between robot and parent frame -->
   <xacro:arg name="xyz" default="0 0 0" />
-  <!-- Rotation offset between robot and parent frame -->
-  <xacro:arg name="rpy" default= "0 0 0" />
-  <!-- Position offset between ee and parent frame -->
-  <xacro:arg name="xyz_ee" default="0 0 0" />
-  <!-- Rotation offset between ee and parent frame -->
-  <xacro:arg name="rpy_ee" default= "0 0 ${-pi/4}" />
-  <!-- Position offset between ee frame and tcp frame -->
-  <xacro:arg name="tcp_xyz" default="0 0 0.1034" />
-  <!-- Rotation offset between ee frame and tcp frame -->
-  <xacro:arg name="tcp_rpy" default="0 0 0" />
-  <!-- Safety distance for the collision capsules -->
-  <xacro:arg name="safety_distance" default="0.03" />
-  <!-- Should self-collision be enabled? -->
-  <xacro:arg name="with_sc" default="false" />
-  <!-- Is the robot being controlled with ros2_control?" -->
-  <xacro:arg name="ros2_control" default="false" />
-  <!-- IP address or hostname of the robot" -->
-  <xacro:arg name="robot_ip" default="" />
-  <!-- Should a fake hardware be used? -->
-  <xacro:arg name="use_fake_hardware" default="false" />
-  <!-- Should fake sensors be used? -->
-  <xacro:arg name="fake_sensor_commands" default="false" />
-  <!-- Should the robot be spawned in Gazebo?" -->
+  <xacro:arg name="rpy" default="0 0 0" />
+  <!-- "none", "franka_default", "rh_p12_rn_a" -->
+  <xacro:arg name="gripper_type" default="franka_default" />
+  <xacro:arg name="parent" default="world" />
+  <xacro:arg name="ros2_control" default="true" />
+  <xacro:arg name="gripper_ros2_control" default="true" />
   <xacro:arg name="gazebo" default="false" />
-  <!-- Should the robot be spawned in Gazebo with effort interfaces?" -->
-  <xacro:arg name="gazebo_effort" default="false" />
-  <!-- Name of the description package -->
-  <xacro:arg name="description_pkg" default="franka_robot_description" />
-  <xacro:arg name="gripper_type" default="franka_default" />
-  <xacro:arg name="use_sim" default="false" />
-  <!-- Append an underscore to the user-provided prefix, if non-empty. -->
+  <xacro:arg name="camera_name" default="zed" />
+  <xacro:arg name="camera_model" default="zedxm" />
+  <xacro:arg name="base_frame"    default="base_link" />
+  <xacro:arg name="cam_pos_x"     default="0.0" />
+  <xacro:arg name="cam_pos_y"     default="0.0" />
+  <xacro:arg name="cam_pos_z"     default="0.0" />
+  <xacro:arg name="cam_roll"      default="0.0" />
+  <xacro:arg name="cam_pitch"     default="0.0" />
+  <xacro:arg name="cam_yaw"       default="0.0" />
+  <xacro:arg name="gnss_frame"    default="" />
+  <!-- ============================================== -->
+  <!-- Property Processing                            -->
+  <!-- ============================================== -->
   <xacro:property name="prefix" value="$(arg arm_prefix)"/>
-  <xacro:property name="modified_prefix" value="${prefix + '_' if prefix else ''}"/>
+  <xacro:property name="modified_prefix" value="${prefix + '_' if prefix != '' else ''}"/>
+  <xacro:property name="use_franka_hand" value="${'true' if '$(arg gripper_type)' == 'franka_default' else 'false'}" />
+  <!-- Include franka_robot macro -->
   <xacro:include filename="$(find franka_robot_description)/robots/common/franka_robot.xacro"/>
-  <!-- <xacro:property name="arg_hand" value="$(arg hand)"/> -->
-  <!-- <xacro:property name="arg_gripper_type" value="$(arg gripper_type)"/> -->
-  <!-- <xacro:property name="load_franka_hand" value="${str(arg_hand).lower() == 'true' and str(arg_gripper_type).lower() == 'default'}"/> -->
-    <!-- Load Franka Robot -->
-  <!-- <xacro:if value="${'$(arg gripper_type)' == 'franka_default'}"> -->
+  <!-- ============================================== -->
+  <!-- Base Robot Arm Instantiation                   -->
+  <!-- ============================================== -->
   <xacro:franka_robot
       arm_id="$(arg arm_id)"
@@ -59,42 +46,43 @@
       dynamics="${xacro.load_yaml('$(find franka_robot_description)/robots/$(arg arm_id)/dynamics.yaml')}"
       gazebo="$(arg gazebo)"
-      hand="$(arg hand)"
-      ee_id="$(arg ee_id)"
-      special_connection="$(arg special_connection)"
-      xyz="$(arg xyz)"
-      rpy="$(arg rpy)"
-      xyz_ee="$(arg xyz_ee)"
-      rpy_ee="$(arg rpy_ee)"
-      tcp_xyz="$(arg tcp_xyz)"
-      tcp_rpy="$(arg tcp_rpy)"
-      safety_distance="$(arg safety_distance)"
-      with_sc="$(arg with_sc)"
-      ros2_control="$(arg ros2_control)"
+      hand="${use_franka_hand}"
+      ee_id="franka_hand"
+      ros2_control="${'true' if '$(arg ros2_control)' == 'true' else 'false'}"
       robot_ip="$(arg robot_ip)"
       use_fake_hardware="$(arg use_fake_hardware)"
       fake_sensor_commands="$(arg fake_sensor_commands)"
-      gazebo_effort="$(arg gazebo_effort)"
-      no_prefix="$(arg no_prefix)"
       arm_prefix="${modified_prefix}"
-      description_pkg="$(arg description_pkg)"
-      connected_to= "base">
+      xyz="$(arg xyz)"
+      rpy="$(arg rpy)"
+      parent="$(arg parent)"
+      connected_to="$(arg parent)">
   </xacro:franka_robot>
-   <!-- </xacro:if> -->
-  <!-- Load RH-P12-RN-A Gripper if selected -->
-  <!-- <xacro:if value="${'$(arg gripper_type)' == 'rh_p12_rn_a' and '$(arg hand)' == 'true'}">
-    <xacro:include filename="$(find robot_dfki_description)/urdf/rh_p12_rn_a/rh_p12_rn_a.xacro" />
-    <xacro:include filename="$(find robot_dfki_description)/gazebo/rh_p12_rn_a/rh_p12_rn_a.gazebo.xacro" />
-    <xacro:include filename="$(find robot_dfki_description)/ros2_control/rh_p12_rn_a/rh_p12_rn_a.ros2_control.xacro" />
-    <joint name="${modified_prefix}rh_p12_rn_base_joint" type="fixed">
-      <parent link="${modified_prefix}$(arg arm_id)_link8"/>
-      <child link="${modified_prefix}rh_p12_rn_base"/>
-      <origin xyz="0 0 0" rpy="0 0 0"/>
-    </joint>
-    <xacro:rh_p12_rn_a prefix="${modified_prefix}" />
-    <xacro:rh_p12_rn_a_gazebo prefix="${modified_prefix}" />
-    <xacro:rh_p12_rn_a_system
-      name="RH-P12-RN-A-System" prefix="${modified_prefix}" use_sim="$(arg use_sim)"
-      use_fake_hardware="$(arg use_fake_hardware)"
-      fake_sensor_commands="$(arg fake_sensor_commands)"/>
-  </xacro:if> -->
+  <!-- ============================================== -->
+  <!-- Dynamic Gripper Attachments                    -->
+  <!-- ============================================== -->
+  <!-- Load Robotis RH-P12-RN-A Gripper if requested -->
+  <xacro:if value="${'$(arg gripper_type)' == 'rh_p12_rn_a'}">
+    <xacro:include filename="$(find franka_robot_description)/urdf/end_effectors/rh_p12_rn_a/rh_p12_rn_a_macro.urdf.xacro"/>
+    <xacro:rh_p12_gripper
+        parent="${modified_prefix}$(arg arm_id)_link8"
+        prefix="${modified_prefix}"
+        use_fake_hardware="$(arg use_fake_hardware)"
+        fake_sensor_commands="$(arg fake_sensor_commands)"
+        ros2_control="$(arg gripper_ros2_control)"
+        use_sim="$(arg use_sim)">
+        <origin xyz="0 0 0.0025" rpy="0 0 -0.785398"/> <!-- adjust rotation if necessary -->
+    </xacro:rh_p12_gripper>
+  </xacro:if>
+  <!-- ============================================== -->
+  <!-- Zed Camera Attachments                    -->
+  <!-- ============================================== -->
+  <xacro:if value="${'$(arg camera_name)' == 'zed'}">
+    <xacro:include filename="$(find franka_robot_description)/urdf/cameras/zed/zed_macro.urdf.xacro" />
+    <xacro:zed_camera name="$(arg camera_name)" model="$(arg camera_model)" parent="${modified_prefix}$(arg arm_id)_link8">
+      <origin
+        xyz="$(arg cam_pos_x) $(arg cam_pos_y) $(arg cam_pos_z)"
+        rpy="$(arg cam_roll) $(arg cam_pitch) $(arg cam_yaw)"
+      />
+    </xacro:zed_camera>
+  </xacro:if>
 </robot>

File: franka_robot_description/urdf/robots/fr3/fr3.urdf.xacro (robot description, xacro)
@@ -1,87 +1,72 @@
 <?xml version='1.0' encoding='utf-8'?>
 <robot xmlns:xacro="http://www.ros.org/wiki/xacro" name="fr3">
-  <!-- ============================================== -->
-  <!-- Arguments provided by franka.launch.py (YAML)  -->
-  <!-- ============================================== -->
-  <xacro:arg name="arm_id" default="fr3" />
+  <xacro:include filename="$(find franka_robot_description)/robots/common/franka_robot.xacro"/>
+  <!-- Define arguments -->
+  <!-- The ID of the robot model to be used -->
+  <xacro:arg name="robot_type" default="fr3" />
+  <!-- The prefix of the robot -->
+  <xacro:arg name="arm_prefix" default="" />
+  <!-- Don't print a prefix for joints, visuals, and links? -->
+  <xacro:arg name="no_prefix" default="false"/>
+  <!-- Should an end-effector be mounted at the flange?" -->
+  <xacro:arg name="hand" default="true" />
+  <!-- Which end-effector would be mounted at the flange?" -->
+  <xacro:arg name="ee_id" default="franka_hand" />
+  <!-- Where is the end-effector connected to, if different from the robot flange?  -->
+  <xacro:arg name="special_connection" default="" />
+  <!-- Position offset between ee and parent frame -->
+  <xacro:arg name="xyz_ee" default="0 0 0" />
+  <!-- Rotation offset between ee and parent frame -->
+  <xacro:arg name="rpy_ee" default= "0 0 ${-pi/4}" />
+  <!-- Position offset between ee frame and tcp frame -->
+  <xacro:arg name="tcp_xyz" default="0 0 0.1034" />
+  <!-- Rotation offset between ee frame and tcp frame -->
+  <xacro:arg name="tcp_rpy" default="0 0 0" />
+  <!-- Safety distance for the collision capsules -->
+  <xacro:arg name="safety_distance" default="0.03" />
+  <!-- Should self-collision be enabled? -->
+  <xacro:arg name="with_sc" default="false" />
+  <!-- Is the robot being controlled with ros2_control?" -->
+  <xacro:arg name="ros2_control" default="false" />
+  <!-- IP address or hostname of the robot" -->
   <xacro:arg name="robot_ip" default="" />
+  <!-- Should a fake hardware be used? -->
   <xacro:arg name="use_fake_hardware" default="false" />
+  <!-- Should fake sensors be used? -->
   <xacro:arg name="fake_sensor_commands" default="false" />
-  <xacro:arg name="use_sim" default="false" />
-  <xacro:arg name="arm_prefix" default="" />
-  <xacro:arg name="xyz" default="0 0 0" />
-  <xacro:arg name="rpy" default="0 0 0" />
-  <!-- "none", "franka_default", "rh_p12_rn_a" -->
-  <xacro:arg name="gripper_type" default="none" />
-  <xacro:arg name="parent" default="world" />
-  <xacro:arg name="ros2_control" default="true" />
-  <xacro:arg name="gripper_ros2_control" default="true" />
+  <!-- Should the robot be spawned in Gazebo?" -->
   <xacro:arg name="gazebo" default="false" />
-  <xacro:arg name="camera_name" default="zed" />
-  <xacro:arg name="camera_model" default="zedxm" />
-  <xacro:arg name="base_frame"    default="base_link" />
-  <xacro:arg name="cam_pos_x"     default="0.0" />
-  <xacro:arg name="cam_pos_y"     default="0.0" />
-  <xacro:arg name="cam_pos_z"     default="0.0" />
-  <xacro:arg name="cam_roll"      default="0.0" />
-  <xacro:arg name="cam_pitch"     default="0.0" />
-  <xacro:arg name="cam_yaw"       default="0.0" />
-  <xacro:arg name="gnss_frame"    default="" />
-  <!-- ============================================== -->
-  <!-- Property Processing                            -->
-  <!-- ============================================== -->
+  <!-- Should the robot be spawned in Gazebo with effort interfaces?" -->
+  <xacro:arg name="gazebo_effort" default="false" />
+  <!-- Name of the description package -->
+  <xacro:arg name="description_pkg" default="franka_robot_description" />
+  <!-- Append an underscore to the user-provided prefix, if non-empty. -->
   <xacro:property name="prefix" value="$(arg arm_prefix)"/>
-  <xacro:property name="modified_prefix" value="${prefix + '_' if prefix != '' else ''}"/>
-  <xacro:property name="use_franka_hand" value="${'true' if '$(arg gripper_type)' == 'franka_default' else 'false'}" />
-  <!-- Include franka_robot macro -->
-  <xacro:include filename="$(find franka_robot_description)/robots/common/franka_robot.xacro"/>
-  <!-- ============================================== -->
-  <!-- Base Robot Arm Instantiation                   -->
-  <!-- ============================================== -->
-  <xacro:franka_robot
-      arm_id="$(arg arm_id)"
-      joint_limits="${xacro.load_yaml('$(find franka_robot_description)/robots/$(arg arm_id)/joint_limits.yaml')}"
-      inertials="${xacro.load_yaml('$(find franka_robot_description)/robots/$(arg arm_id)/inertials.yaml')}"
-      kinematics="${xacro.load_yaml('$(find franka_robot_description)/robots/$(arg arm_id)/kinematics.yaml')}"
-      dynamics="${xacro.load_yaml('$(find franka_robot_description)/robots/$(arg arm_id)/dynamics.yaml')}"
-      gazebo="$(arg gazebo)"
-      hand="${use_franka_hand}"
-      ee_id="franka_hand"
-      ros2_control="${'true' if '$(arg ros2_control)' == 'true' else 'false'}"
-      robot_ip="$(arg robot_ip)"
-      use_fake_hardware="$(arg use_fake_hardware)"
-      fake_sensor_commands="$(arg fake_sensor_commands)"
-      arm_prefix="${modified_prefix}"
-      xyz="$(arg xyz)"
-      rpy="$(arg rpy)"
-      parent="$(arg parent)"
-      connected_to="$(arg parent)">
+  <xacro:property name="modified_prefix" value="${prefix + '_' if prefix else ''}"/>
+  <xacro:franka_robot robot_type="fr3"
+                      joint_limits="${xacro.load_yaml('$(find franka_robot_description)/robots/fr3/joint_limits.yaml')}"
+                      inertials="${xacro.load_yaml('$(find franka_robot_description)/robots/fr3/inertials.yaml')}"
+                      kinematics="${xacro.load_yaml('$(find franka_robot_description)/robots/fr3/kinematics.yaml')}"
+                      accelerometer_config="${xacro.load_yaml('$(find franka_robot_description)/robots/fr3/accelerometers.yaml')}"
+                      dynamics="${xacro.load_yaml('$(find franka_robot_description)/robots/fr3/dynamics.yaml')}"
+                      gazebo="$(arg gazebo)"
+                      hand="$(arg hand)"
+                      ee_id="$(arg ee_id)"
+                      special_connection="$(arg special_connection)"
+                      xyz_ee="$(arg xyz_ee)"
+                      rpy_ee="$(arg rpy_ee)"
+                      tcp_xyz="$(arg tcp_xyz)"
+                      tcp_rpy="$(arg tcp_rpy)"
+                      safety_distance="$(arg safety_distance)"
+                      with_sc="$(arg with_sc)"
+                      ros2_control="$(arg ros2_control)"
+                      robot_ip="$(arg robot_ip)"
+                      use_fake_hardware="$(arg use_fake_hardware)"
+                      fake_sensor_commands="$(arg fake_sensor_commands)"
+                      gazebo_effort="$(arg gazebo_effort)"
+                      no_prefix="$(arg no_prefix)"
+                      arm_prefix="${modified_prefix}"
+                      description_pkg="$(arg description_pkg)"
+                      connected_to= "base">
   </xacro:franka_robot>
-  <!-- ============================================== -->
-  <!-- Dynamic Gripper Attachments                    -->
-  <!-- ============================================== -->
-  <!-- TODO: move it to bimanual_dfki.urdf.xacro -->
-  <!-- Load Robotis RH-P12-RN-A Gripper if requested -->
-  <xacro:if value="${'$(arg gripper_type)' == 'rh_p12_rn_a'}">
-    <xacro:include filename="$(find franka_robot_description)/urdf/end_effectors/rh_p12_rn_a/rh_p12_rn_a_macro.urdf.xacro"/>
-    <xacro:rh_p12_gripper
-        parent="${modified_prefix}$(arg arm_id)_link8"
-        prefix="${modified_prefix}"
-        use_fake_hardware="$(arg use_fake_hardware)"
-        fake_sensor_commands="$(arg fake_sensor_commands)"
-        ros2_control="$(arg gripper_ros2_control)"
-        use_sim="$(arg use_sim)">
-        <origin xyz="0 0 0.0025" rpy="0 0 -0.785398"/> <!-- adjust rotation if necessary -->
-    </xacro:rh_p12_gripper>
-  </xacro:if>
-  <!-- TODO: move it to bimanual_dfki.urdf.xacro -->
-  <xacro:if value="${'$(arg camera_name)' == 'zed'}">
-    <xacro:include filename="$(find franka_robot_description)/urdf/cameras/zed/zed_macro.urdf.xacro" />
-    <xacro:zed_camera name="$(arg camera_name)" model="$(arg camera_model)" parent="${modified_prefix}$(arg arm_id)_link8">
-      <origin
-        xyz="$(arg cam_pos_x) $(arg cam_pos_y) $(arg cam_pos_z)"
-        rpy="$(arg cam_roll) $(arg cam_pitch) $(arg cam_yaw)"
-      />
-    </xacro:zed_camera>
-  </xacro:if>
 </robot>
