Commit message: adjust to the old version of the description

File: franka_robot_description/robots/common/utils.xacro (robot description, xacro)
@@ -32,16 +32,16 @@
   <!-- self_collision_geometries:  self <collision> models        -->
   <!-- ========================================================== -->
-  <xacro:macro name="link_with_sc" params="name no_prefix:='false' rpy:='0 0 0' **self_collision_geometries gazebo:=false with_sc:=false with_accelerometers:=false">
-    <xacro:property name="prefix" value="${'' if no_prefix else arm_prefix + robot_type + '_'}" />
+  <xacro:macro name="link_with_sc" params="name no_prefix:='false' rpy:='0 0 0' **self_collision_geometries gazebo:=false with_sc:=false">
+    <xacro:property name="prefix" value="${'' if no_prefix else arm_prefix + arm_id + '_'}" />
     <!-- sub-link defining detailed meshes for collision with environment -->
     <link name="${prefix}${name}">
       <visual name="${prefix}${name}_visual">
         <geometry>
-          <mesh filename="package://${description_pkg}/meshes/robots/${robot_type}/visual/${name}.dae" />
+          <mesh filename="package://${description_pkg}/meshes/robot_arms/${arm_id}/visual/${name}.dae" />
         </geometry>
       </visual>
       <collision name="${prefix}${name}_collision">
         <geometry>
-          <mesh filename="package://franka_description/meshes/robots/${robot_type}/collision/${name}.stl" />
+          <mesh filename="package://franka_description/meshes/robot_arms/${arm_id}/collision/${name}.stl" />
         </geometry>
       </collision>
@@ -61,7 +61,4 @@
         <child link="${prefix}${name}_sc" />
       </joint>
-    </xacro:if>
-    <xacro:if value="${with_accelerometers}">
-      <xacro:franka-accelerometers prefix="${prefix}" name="${name}" config="${accelerometer_config}" />
     </xacro:if>
   </xacro:macro>
@@ -157,23 +154,23 @@
   <!-- when simulating with franka_hw_sim plugin                  -->
   <!--                                                            -->
-  <!-- robot_type - Arm ID of the fer to simulate (default 'fer')     -->
-  <!-- ========================================================== -->
-  <xacro:macro name="transmission-franka-state" params="robot_type:=fer">
-    <transmission name="${arm_prefix}${robot_type}_franka_state">
+  <!-- arm_id - Arm ID of the fer to simulate (default 'fer')     -->
+  <!-- ========================================================== -->
+  <xacro:macro name="transmission-franka-state" params="arm_id:=fer">
+    <transmission name="${arm_prefix}${arm_id}_franka_state">
       <type>franka_hw/FrankaStateInterface</type>
-      <joint name="${arm_prefix}${robot_type}_joint1"><hardwareInterface>franka_hw/FrankaStateInterface</hardwareInterface></joint>
-      <joint name="${arm_prefix}${robot_type}_joint2"><hardwareInterface>franka_hw/FrankaStateInterface</hardwareInterface></joint>
-      <joint name="${arm_prefix}${robot_type}_joint3"><hardwareInterface>franka_hw/FrankaStateInterface</hardwareInterface></joint>
-      <joint name="${arm_prefix}${robot_type}_joint4"><hardwareInterface>franka_hw/FrankaStateInterface</hardwareInterface></joint>
-      <joint name="${arm_prefix}${robot_type}_joint5"><hardwareInterface>franka_hw/FrankaStateInterface</hardwareInterface></joint>
-      <joint name="${arm_prefix}${robot_type}_joint6"><hardwareInterface>franka_hw/FrankaStateInterface</hardwareInterface></joint>
-      <joint name="${arm_prefix}${robot_type}_joint7"><hardwareInterface>franka_hw/FrankaStateInterface</hardwareInterface></joint>
-      <actuator name="${arm_prefix}${robot_type}_motor1"><hardwareInterface>franka_hw/FrankaStateInterface</hardwareInterface></actuator>
-      <actuator name="${arm_prefix}${robot_type}_motor2"><hardwareInterface>franka_hw/FrankaStateInterface</hardwareInterface></actuator>
-      <actuator name="${arm_prefix}${robot_type}_motor3"><hardwareInterface>franka_hw/FrankaStateInterface</hardwareInterface></actuator>
-      <actuator name="${arm_prefix}${robot_type}_motor4"><hardwareInterface>franka_hw/FrankaStateInterface</hardwareInterface></actuator>
-      <actuator name="${arm_prefix}${robot_type}_motor5"><hardwareInterface>franka_hw/FrankaStateInterface</hardwareInterface></actuator>
-      <actuator name="${arm_prefix}${robot_type}_motor6"><hardwareInterface>franka_hw/FrankaStateInterface</hardwareInterface></actuator>
-      <actuator name="${arm_prefix}${robot_type}_motor7"><hardwareInterface>franka_hw/FrankaStateInterface</hardwareInterface></actuator>
+      <joint name="${arm_prefix}${arm_id}_joint1"><hardwareInterface>franka_hw/FrankaStateInterface</hardwareInterface></joint>
+      <joint name="${arm_prefix}${arm_id}_joint2"><hardwareInterface>franka_hw/FrankaStateInterface</hardwareInterface></joint>
+      <joint name="${arm_prefix}${arm_id}_joint3"><hardwareInterface>franka_hw/FrankaStateInterface</hardwareInterface></joint>
+      <joint name="${arm_prefix}${arm_id}_joint4"><hardwareInterface>franka_hw/FrankaStateInterface</hardwareInterface></joint>
+      <joint name="${arm_prefix}${arm_id}_joint5"><hardwareInterface>franka_hw/FrankaStateInterface</hardwareInterface></joint>
+      <joint name="${arm_prefix}${arm_id}_joint6"><hardwareInterface>franka_hw/FrankaStateInterface</hardwareInterface></joint>
+      <joint name="${arm_prefix}${arm_id}_joint7"><hardwareInterface>franka_hw/FrankaStateInterface</hardwareInterface></joint>
+      <actuator name="${arm_prefix}${arm_id}_motor1"><hardwareInterface>franka_hw/FrankaStateInterface</hardwareInterface></actuator>
+      <actuator name="${arm_prefix}${arm_id}_motor2"><hardwareInterface>franka_hw/FrankaStateInterface</hardwareInterface></actuator>
+      <actuator name="${arm_prefix}${arm_id}_motor3"><hardwareInterface>franka_hw/FrankaStateInterface</hardwareInterface></actuator>
+      <actuator name="${arm_prefix}${arm_id}_motor4"><hardwareInterface>franka_hw/FrankaStateInterface</hardwareInterface></actuator>
+      <actuator name="${arm_prefix}${arm_id}_motor5"><hardwareInterface>franka_hw/FrankaStateInterface</hardwareInterface></actuator>
+      <actuator name="${arm_prefix}${arm_id}_motor6"><hardwareInterface>franka_hw/FrankaStateInterface</hardwareInterface></actuator>
+      <actuator name="${arm_prefix}${arm_id}_motor7"><hardwareInterface>franka_hw/FrankaStateInterface</hardwareInterface></actuator>
     </transmission>
   </xacro:macro>
@@ -182,10 +179,10 @@
   <!-- when simulating with franka_hw_sim plugin                    -->
   <!--                                                              -->
-  <!-- robot_type - Arm ID of the fer to simulate (default 'fer')       -->
+  <!-- arm_id - Arm ID of the fer to simulate (default 'fer')       -->
   <!-- root   - Joint name of the base of the robot                 -->
   <!-- tip    - Joint name of the tip of the robot (flange or hand) -->
   <!-- ============================================================ -->
-  <xacro:macro name="transmission-franka-model" params="robot_type:=fer root:=fer_joint1 tip:=fer_joint7">
-    <transmission name="${arm_prefix}${robot_type}_franka_model">
+  <xacro:macro name="transmission-franka-model" params="arm_id:=fer root:=fer_joint1 tip:=fer_joint7">
+    <transmission name="${arm_prefix}${arm_id}_franka_model">
       <type>franka_hw/FrankaModelInterface</type>
       <joint name="${root}">
@@ -226,9 +223,4 @@
                          soft_lower_limit="${limits.lower}"
                          soft_upper_limit="${limits.upper}" />
-      <!-- Add position-based velocity limits if they exist -->
-      <xacro:if value="${'position_based_velocity_limits' in config[name]}">
-        <xacro:property name="position_based_velocity_limits" value="${config[name]['position_based_velocity_limits']}" lazy_eval="false" />
-        <position_based_velocity_limits velocity_offset="${position_based_velocity_limits.velocity_offset}" deceleration_limit="${position_based_velocity_limits.deceleration_limit}" />
-      </xacro:if>
   </xacro:macro>
   <!-- ========================================================================= -->
@@ -258,30 +250,3 @@
              xyz="${kinematics.x} ${kinematics.y} ${kinematics.z}" />
   </xacro:macro>
-  <!-- ================================================================================== -->
-  <!-- Adds the accelerometer frames given a config file of link accelerometers           -->
-  <!--                                                                                    -->
-  <!-- name   - Name of the link for which to add accelerometers to                       -->
-  <!-- prefix - Prefix to name                                                            -->
-  <!-- config - YAML struct defining link accelerometers (e.g. fr3v2/accelerometers.yaml) -->
-  <!-- ================================================================================== -->
-  <xacro:macro name="franka-accelerometers" params="name prefix config">
-      <xacro:property name="accelerometer_top" value="${config[name]['accelerometer_top']}" lazy_eval="false" />
-      <xacro:property name="accelerometer_bottom" value="${config[name]['accelerometer_bottom']}" lazy_eval="false" />
-      <link name="${prefix}${name}_accelerometer_top">
-      </link>
-      <joint name="${prefix}${name}_accelerometer_top_joint" type="fixed">
-        <origin rpy="${accelerometer_top.roll} ${accelerometer_top.pitch} ${accelerometer_top.yaw}"
-             xyz="${accelerometer_top.x} ${accelerometer_top.y} ${accelerometer_top.z}" />
-        <parent link="${prefix}${name}" />
-        <child link="${prefix}${name}_accelerometer_top" />
-      </joint>
-      <link name="${prefix}${name}_accelerometer_bottom">
-      </link>
-      <joint name="${prefix}${name}_accelerometer_bottom_joint" type="fixed">
-        <origin rpy="${accelerometer_bottom.roll} ${accelerometer_bottom.pitch} ${accelerometer_bottom.yaw}"
-             xyz="${accelerometer_bottom.x} ${accelerometer_bottom.y} ${accelerometer_bottom.z}" />
-        <parent link="${prefix}${name}" />
-        <child link="${prefix}${name}_accelerometer_bottom" />
-      </joint>
-  </xacro:macro>
 </robot>

File: franka_robot_description/robots/fr3/fr3.srdf.xacro (robot description, xacro)
@@ -2,6 +2,10 @@
 <robot xmlns:xacro="http://www.ros.org/wiki/xacro" name="fr3">
   <xacro:include filename="$(find franka_description)/robots/common/franka_arm.srdf.xacro"/>
-  <!-- The ID of the robot model to be used -->
-  <xacro:arg name="robot_type" default="fr3" />
+  <!--
+    DEPRECATION NOTICE
+    argument arm_id is no longer supported and will be removed in the future.
+    This argument is ignored.
+  -->
+  <xacro:arg name="arm_id" default="fr3" />
   <!-- The prefix of the robot -->
   <xacro:arg name="arm_prefix" default="" />
@@ -12,5 +16,5 @@
   <!-- Which end-effector would be mounted at the flange?" -->
   <xacro:arg name="ee_id" default="franka_hand" />
-  <xacro:franka_arm_srdf robot_type="$(arg robot_type)"
+  <xacro:franka_arm_srdf arm_id="$(arg arm_id)"
                       hand="$(arg hand)"
                       ee_id="$(arg ee_id)"

File: franka_robot_description/robots/fr3/fr3.urdf.xacro (robot description, xacro)
@@ -2,7 +2,10 @@
 <robot xmlns:xacro="http://www.ros.org/wiki/xacro" name="fr3">
   <xacro:include filename="$(find franka_description)/robots/common/franka_robot.xacro"/>
-  <!-- Define arguments -->
-  <!-- The ID of the robot model to be used -->
-  <xacro:arg name="robot_type" default="fr3" />
+  <!--
+    DEPRECATION NOTICE
+    argument arm_id is no longer supported and will be removed in the future.
+    This argument is ignored.
+  -->
+  <xacro:arg name="arm_id" default="fr3" />
   <!-- The prefix of the robot -->
   <xacro:arg name="arm_prefix" default="" />
@@ -15,4 +18,8 @@
   <!-- Where is the end-effector connected to, if different from the robot flange?  -->
   <xacro:arg name="special_connection" default="" />
+  <!-- Position offset between robot and parent frame -->
+  <xacro:arg name="xyz" default="0 0 0" />
+  <!-- Rotation offset between robot and parent frame -->
+  <xacro:arg name="rpy" default= "0 0 0" />
   <!-- Position offset between ee and parent frame -->
   <xacro:arg name="xyz_ee" default="0 0 0" />
@@ -44,9 +51,8 @@
   <xacro:property name="prefix" value="$(arg arm_prefix)"/>
   <xacro:property name="modified_prefix" value="${prefix + '_' if prefix else ''}"/>
-  <xacro:franka_robot robot_type="fr3"
+  <xacro:franka_robot arm_id="fr3"
                       joint_limits="${xacro.load_yaml('$(find franka_description)/robots/fr3/joint_limits.yaml')}"
                       inertials="${xacro.load_yaml('$(find franka_description)/robots/fr3/inertials.yaml')}"
                       kinematics="${xacro.load_yaml('$(find franka_description)/robots/fr3/kinematics.yaml')}"
-                      accelerometer_config="${xacro.load_yaml('$(find franka_description)/robots/fr3/accelerometers.yaml')}"
                       dynamics="${xacro.load_yaml('$(find franka_description)/robots/fr3/dynamics.yaml')}"
                       gazebo="$(arg gazebo)"
@@ -54,4 +60,6 @@
                       ee_id="$(arg ee_id)"
                       special_connection="$(arg special_connection)"
+                      xyz="$(arg xyz)"
+                      rpy="$(arg rpy)"
                       xyz_ee="$(arg xyz_ee)"
                       rpy_ee="$(arg rpy_ee)"

Commit message: add working franka left (without gipper controller)

File: franka_robot_description/robots/common/franka_arm.ros2_control.xacro (robot description, xacro)
@@ -58,5 +58,5 @@
       <xacro:configure_joint joint_name="${arm_prefix}${arm_id}_joint6" initial_position="${pi/2}"/>
       <xacro:configure_joint joint_name="${arm_prefix}${arm_id}_joint7" initial_position="${pi/4}"/>
-      <xacro:if value="${gazebo and hand}">
+      <xacro:if value="${(gazebo or use_fake_hardware) and hand}">
         <xacro:configure_joint joint_name="${arm_prefix}${arm_id}_finger_joint1" initial_position="0.0" />
       </xacro:if>

File: franka_robot_description/urdf/end_effectors/rh_p12_rn_a/rh_p12_rn_a.ros2_control.xacro (robot description, xacro)
@@ -1,5 +1,5 @@
 <?xml version="1.0"?>
 <robot xmlns:xacro="http://www.ros.org/wiki/xacro">
-  <xacro:macro name="rh_p12_rn_a_system" params="name prefix port_name:=^|/dev/ttyUSB0 use_sim:=^|false use_fake_hardware:=^|false fake_sensor_commands:=^|false">
+  <xacro:macro name="rh_p12_rn_a_system" params="name prefix port_name:=^|/dev/ttyUSB1 use_sim:=^|false use_fake_hardware:=^|false fake_sensor_commands:=^|false">
     <ros2_control name="${name}" type="system" is_async="true">
       <xacro:if value="${use_sim}">

File: franka_robot_description/urdf/main_assemblies/bimanual_dfki.urdf.xacro (robot description, xacro)
@@ -12,4 +12,6 @@
   <xacro:arg name="xyz" default="0 0 0" />
   <xacro:arg name="rpy" default="0 0 0" />
+  <xacro:arg name="xyz_ee" default="0 0 0" />
+  <xacro:arg name="rpy_ee" default="0 0 0" />
   <!-- "none", "franka_default", "rh_p12_rn_a" -->
   <xacro:arg name="gripper_type" default="franka_default" />
@@ -55,4 +57,6 @@
       xyz="$(arg xyz)"
       rpy="$(arg rpy)"
+      xyz_ee="$(arg xyz_ee)"
+      rpy_ee="$(arg rpy_ee)"
       parent="$(arg parent)"
       connected_to="$(arg parent)">
@@ -71,5 +75,5 @@
         ros2_control="$(arg gripper_ros2_control)"
         use_sim="$(arg use_sim)">
-        <origin xyz="0 0 0.0025" rpy="0 0 -0.785398"/> <!-- adjust rotation if necessary -->
+        <origin xyz="$(arg xyz_ee)" rpy="$(arg rpy_ee)"/>
     </xacro:rh_p12_gripper>
   </xacro:if>
@@ -77,5 +81,5 @@
   <!-- Zed Camera Attachments                    -->
   <!-- ============================================== -->
-  <xacro:if value="${'$(arg camera_name)' == 'zed'}">
+  <xacro:if value="${'$(arg camera_name)' == 'zed' and '$(arg gripper_type)' == 'rh_p12_rn_a'}">
     <xacro:include filename="$(find franka_robot_description)/urdf/cameras/zed/zed_macro.urdf.xacro" />
     <xacro:zed_camera name="$(arg camera_name)" model="$(arg camera_model)" parent="${modified_prefix}$(arg arm_id)_link8">
