Commit message: Save current chenges

File: franka_robot_description/urdf/end_effectors/rh_p12_rn_a/rh_p12_rn_a.xacro (robot description, xacro)
@@ -25,5 +25,5 @@
       <inertial>
         <origin xyz="0.000 0.000 0.032" rpy="0 0 0"/>
-        <mass value="0.436"/>
+        <mass value="0.336"/>  <!--+100g for cabeling: orig: 0.236-->
         <inertia ixx="0.000001" ixy="0.0" ixz="0.0" iyy="0.000001" iyz="0.0" izz="0.000001" />
       </inertial>

File: franka_robot_description/urdf/robots/fr3/fr3.urdf.xacro (robot description, xacro)
@@ -18,4 +18,14 @@
   <xacro:arg name="gripper_ros2_control" default="true" />
   <xacro:arg name="gazebo" default="false" />
+  <xacro:arg name="camera_name" default="zed" />
+  <xacro:arg name="camera_model" default="zedxm" />
+  <xacro:arg name="base_frame"    default="base_link" />
+  <xacro:arg name="cam_pos_x"     default="0.0" />
+  <xacro:arg name="cam_pos_y"     default="0.0" />
+  <xacro:arg name="cam_pos_z"     default="0.0" />
+  <xacro:arg name="cam_roll"      default="0.0" />
+  <xacro:arg name="cam_pitch"     default="0.0" />
+  <xacro:arg name="cam_yaw"       default="0.0" />
+  <xacro:arg name="gnss_frame"    default="" />
   <!-- ============================================== -->
   <!-- Property Processing                            -->
@@ -51,4 +61,5 @@
   <!-- Dynamic Gripper Attachments                    -->
   <!-- ============================================== -->
+  <!-- TODO: move it to bimanual_dfki.urdf.xacro -->
   <!-- Load Robotis RH-P12-RN-A Gripper if requested -->
   <xacro:if value="${'$(arg gripper_type)' == 'rh_p12_rn_a'}">
@@ -61,6 +72,16 @@
         ros2_control="$(arg gripper_ros2_control)"
         use_sim="$(arg use_sim)">
-        <origin xyz="0 0 0" rpy="0 0 -0.785398"/> <!-- adjust rotation if necessary -->
+        <origin xyz="0 0 0.0025" rpy="0 0 -0.785398"/> <!-- adjust rotation if necessary -->
     </xacro:rh_p12_gripper>
   </xacro:if>
+  <!-- TODO: move it to bimanual_dfki.urdf.xacro -->
+  <xacro:if value="${'$(arg camera_name)' == 'zed'}">
+    <xacro:include filename="$(find franka_robot_description)/urdf/cameras/zed/zed_macro.urdf.xacro" />
+    <xacro:zed_camera name="$(arg camera_name)" model="$(arg camera_model)" parent="${modified_prefix}$(arg arm_id)_link8">
+      <origin
+        xyz="$(arg cam_pos_x) $(arg cam_pos_y) $(arg cam_pos_z)"
+        rpy="$(arg cam_roll) $(arg cam_pitch) $(arg cam_yaw)"
+      />
+    </xacro:zed_camera>
+  </xacro:if>
 </robot>

Commit message: add a new frame

File: franka_robot_description/urdf/end_effectors/rh_p12_rn_a/rh_p12_rn_a.xacro (robot description, xacro)
@@ -29,4 +29,12 @@
       </inertial>
     </link>
+    <!-- Grasp Point Joint -->
+    <joint name="${prefix}rh_p12_rn_grasp_point_joint" type="fixed">
+      <parent link="${prefix}rh_p12_rn_base"/>
+      <child link="${prefix}rh_p12_rn_grasp_point"/>
+      <origin xyz="0 0 0.10" rpy="0 0 0"/>
+    </joint>
+    <!-- Grasp Point Link -->
+    <link name="${prefix}rh_p12_rn_grasp_point"/>
     <!-- Joint -->
     <joint name="${prefix}rh_r1" type="revolute">
